Commit message: Implementación de navegación autónoma Nav2, AMCL y mapas del laberinto

File: urdf/gazebo/gazebo_plugins.xacro (robot description, xacro)
@@ -14,9 +14,9 @@
             <!-- Nombres de tópicos corregidos para Ignition -->
             <topic>cmd_vel</topic>
-            <odom_topic>model/tretabot/odometry</odom_topic>
-            <tf_topic>model/tretabot/tf</tf_topic>
+            <odom_topic>model/tetrabot/odometry</odom_topic>
+            <tf_topic>model/tetrabot/tf</tf_topic>
             <!-- Coincidiendo con tu Launch prefix -->
-            <frame_id>tretabot/odom</frame_id>
-            <child_frame_id>tretabot/base_footprint</child_frame_id>
+            <frame_id>tetrabot/odom</frame_id>
+            <child_frame_id>tetrabot/base_footprint</child_frame_id>
             <odom_publisher_frequency>30</odom_publisher_frequency>
             <max_linear_acceleration>0.5</max_linear_acceleration>
@@ -41,22 +41,28 @@
 <!-- =========== Lidar Sensor ============ -->
     <gazebo reference="lidar_link">
-        <sensor name='gpu_lidar' type='gpu_lidar'>
+        <sensor name='gpu_lidar' type='gpu_lidar'>"
             <pose relative_to='lidar_link'>0 0 0 0 0 0</pose>
             <topic>scan</topic>
-            <update_rate>10</update_rate> <always_on>1</always_on>
+            <update_rate>2</update_rate>
+            <always_on>1</always_on>
             <visualize>1</visualize>
             <lidar>
                 <scan>
                     <horizontal>
-                        <samples>360</samples>
+                        <samples>640</samples>
                         <resolution>1</resolution>
-                        <min_angle>-3.14159265</min_angle> <max_angle>3.14159265</max_angle>
+                        <min_angle>-1.396263</min_angle>
+                        <max_angle>1.396263</max_angle>
                     </horizontal>
-                    <vertical>
-                        <samples>16</samples> <resolution>1</resolution>
-                        <min_angle>-0.261799</min_angle> <max_angle>0.261799</max_angle>  </vertical>
+                    <!--<vertical> Not needed if not scanning vertically
+                        <samples>1</samples>
+                        <resolution>0.01</resolution>
+                        <min_angle>0</min_angle>
+                        <max_angle>0</max_angle>
+                    </vertical>-->
                 </scan>
                 <range>
-                    <min>0.10</min> <max>10.0</max>
+                    <min>0.08</min>
+                    <max>10.0</max>
                     <resolution>0.01</resolution>
                 </range>
@@ -64,5 +70,5 @@
                     <type>gaussian</type>
                     <mean>0.0</mean>
-                    <stddev>0.01</stddev>
+                    <stddev>0.001</stddev>
                 </noise>
             </lidar>
@@ -99,3 +105,32 @@
     </gazebo>
 <!--=========================================-->
+<gazebo reference="faro_link">
+  <visual>
+    <material>
+      <ambient>1 1 0 1</ambient>
+      <diffuse>1 1 0 1</diffuse>
+      <specular>1 1 1 1</specular>
+      <emissive>1 1 0 1</emissive> <!-- Esto hace que el faro brille en la simulación -->
+    </material>
+  </visual>
+  <!-- Luz puntual que emite el faro -->
+  <light name="faro_luz" type="spot">
+    <pose>0 0 0 0 0 0</pose>
+    <diffuse>1 1 1 1</diffuse>
+    <specular>.1 .1 .1 1</specular>
+    <attenuation>
+      <range>10</range>
+      <constant>0.5</constant>
+      <linear>0.01</linear>
+      <quadratic>0.001</quadratic>
+    </attenuation>
+    <direction>1 0 0</direction> <!-- Hacia adelante -->
+    <spot>
+      <inner_angle>0.1</inner_angle>
+      <outer_angle>0.5</outer_angle>
+      <falloff>1.2</falloff>
+    </spot>
+    <cast_shadows>true</cast_shadows>
+  </light>
+</gazebo>
 </robot>

File: urdf/gazebo/gazebo_properties.xacro (robot description, xacro)
@@ -13,4 +13,24 @@
   </gazebo>
   <gazebo reference="camara_link">
+    <mu1 value="0.5"/> <!-- Friction coefficient in the first direction -->
+    <mu2 value="0.5"/> <!-- Friction coefficient in the second direction -->
+  </gazebo>
+  <gazebo reference="faro_link">
+    <mu1 value="0.5"/> <!-- Friction coefficient in the first direction -->
+    <mu2 value="0.5"/> <!-- Friction coefficient in the second direction -->
+  </gazebo>
+  <gazebo reference="antena_link">
+    <mu1 value="0.5"/> <!-- Friction coefficient in the first direction -->
+    <mu2 value="0.5"/> <!-- Friction coefficient in the second direction -->
+  </gazebo>
+  <gazebo reference="ultrasonico_der_link">
+    <mu1 value="0.5"/> <!-- Friction coefficient in the first direction -->
+    <mu2 value="0.5"/> <!-- Friction coefficient in the second direction -->
+  </gazebo>
+  <gazebo reference="ultrasonico_iz_link">
+    <mu1 value="0.5"/> <!-- Friction coefficient in the first direction -->
+    <mu2 value="0.5"/> <!-- Friction coefficient in the second direction -->
+  </gazebo>
+  <gazebo reference="ultrasonico_tra_link">
     <mu1 value="0.5"/> <!-- Friction coefficient in the first direction -->
     <mu2 value="0.5"/> <!-- Friction coefficient in the second direction -->

File: urdf/modules/base_y_llantas.xacro (robot description, xacro)
@@ -14,7 +14,7 @@
   <link name="base_link">
     <inertial>
-      <origin xyz="0.0112256 -0 0.0778907" rpy="0 0 0"/>
-      <mass value="4.81654"/>
-      <inertia ixx="0.0259231" ixy="0" ixz="-0.00401137" iyy="0.0296606" iyz="0" izz="0.0400591"/>
+      <origin xyz="0.0107572 -0.000338235 0.0779814" rpy="0 0 0"/>
+      <mass value="4.83557"/>
+      <inertia ixx="0.0260829" ixy="-0.000213984" ixz="-0.00395219" iyy="0.0299972" iyz="3.98093e-05" izz="0.0405276"/>
     </inertial>
     <!-- Part base_t -->
@@ -38,11 +38,11 @@
   <link name="llanta_dere_del_link">
     <inertial>
-      <origin xyz="0 -0 -0.0264625" rpy="0 0 0"/>
+      <origin xyz="-0 -0 -0.0264625" rpy="0 0 0"/>
       <mass value="0.0901579"/>
-      <inertia ixx="2.81915e-05" ixy="0" ixz="0" iyy="2.83576e-05" iyz="0" izz="4.79296e-05"/>
+      <inertia ixx="2.81915e-05" ixy="0" ixz="0" iyy="2.83576e-05" iyz="-0" izz="4.79296e-05"/>
     </inertial>
     <!-- Part llanta_dere_del -->
     <visual>
-      <origin xyz="0 0 -0.015" rpy="1.5708 -0 0"/>
+      <origin xyz="-0 0 -0.015" rpy="1.5708 0 0"/>
       <geometry>
         <mesh filename="package://my_robot_description/assets/llanta_dere_del.stl"/>
@@ -53,5 +53,5 @@
     </visual>
     <collision>
-      <origin xyz="0 0 -0.015" rpy="1.5708 -0 0"/>
+      <origin xyz="-0 0 -0.015" rpy="1.5708 0 0"/>
       <geometry>
         <mesh filename="package://my_robot_description/assets/llanta_dere_del.stl"/>
@@ -61,5 +61,5 @@
   <!-- Joint from base_t to llanta_dere_del -->
   <joint name="llanta_dere_del_joint" type="continuous">
-    <origin xyz="0.0441 -0.095 0.0162" rpy="-1.5708 -0 0"/>
+    <origin xyz="0.0441 -0.095 0.0162" rpy="-1.5708 0.765592 0"/>
     <parent link="base_link"/>
     <child link="llanta_dere_del_link"/>

File: urdf/modules/camara.xacro (robot description, xacro)
@@ -6,20 +6,20 @@
   <link name="camara_link">
     <inertial>
-      <origin xyz="0 0 -0.00772686" rpy="0 0 0"/>
-      <mass value="0.0784361"/>
-      <inertia ixx="2.01766e-05" ixy="0" ixz="0" iyy="2.01766e-05" iyz="0" izz="3.18165e-05"/>
+      <origin xyz="-0 0 -0.00516528" rpy="0 0 0"/>
+      <mass value="0.0399941"/>
+      <inertia ixx="6.59521e-06" ixy="0" ixz="0" iyy="6.59521e-06" iyz="0" izz="1.04207e-05"/>
     </inertial>
     <!-- Part camara_t_s -->
     <visual>
-      <origin xyz="-0 0 0.005" rpy="1.5708 1.5708 0"/>
+      <origin xyz="-0 0 0.005" rpy="3.14159 -0 1.5708"/>
       <geometry>
         <mesh filename="package://my_robot_description/assets/camara_t_s.stl"/>
       </geometry>
       <material name="camara_t_s_material">
-        <color rgba="0.439216 0.47451 0.501961 1"/>
+        <color rgba="0.262745 0.282353 0.301961 1"/>
       </material>
     </visual>
     <collision>
-      <origin xyz="-0 0 0.005" rpy="1.5708 1.5708 0"/>
+      <origin xyz="-0 0 0.005" rpy="3.14159 -0 1.5708"/>
       <geometry>
         <mesh filename="package://my_robot_description/assets/camara_t_s.stl"/>
@@ -29,5 +29,5 @@
   <!-- Joint from base_t to camara_t_s -->
   <joint name="camara_joint" type="fixed">
-    <origin xyz="0.115 0 0.135" rpy="0 0 0"/>
+    <origin xyz="0.115 0 0.135" rpy=" 0 0 0 "/>
     <parent link="base_link"/>
     <child link="camara_link"/>

File: urdf/modules/lidar.xacro (robot description, xacro)
@@ -3,8 +3,8 @@
 <!-- Onshape document_id: 3023829f8e4e5c564f6b4985 -->
 <robot xmlns:xacro="http://www.ros.org/wiki/xacro">
-  <!-- Link lidar_t_s -->
+<!-- Link lidar_t_s -->
   <link name="lidar_link">
     <inertial>
-      <origin xyz="-0 -0 -0.00994579" rpy="0 0 0"/>
+      <origin xyz="-0 0 -0.00994579" rpy="0 0 0"/>
       <mass value="0.0591873"/>
       <inertia ixx="1.18545e-05" ixy="0" ixz="0" iyy="1.18545e-05" iyz="0" izz="1.49382e-05"/>
@@ -12,5 +12,5 @@
     <!-- Part lidar_t_s -->
     <visual>
-      <origin xyz="0 -0 0.005" rpy="3.14159 -0 0"/>
+      <origin xyz="0 0 0.005" rpy="3.14159 -0 0"/>
       <geometry>
         <mesh filename="package://my_robot_description/assets/lidar_t_s.stl"/>
@@ -21,5 +21,5 @@
     </visual>
     <collision>
-      <origin xyz="0 -0 0.005" rpy="3.14159 -0 0"/>
+      <origin xyz="0 0 0.005" rpy="3.14159 -0 0"/>
       <geometry>
         <mesh filename="package://my_robot_description/assets/lidar_t_s.stl"/>
@@ -29,5 +29,5 @@
   <!-- Joint from base_t to lidar_t_s -->
   <joint name="lidar_joint" type="fixed">
-    <origin xyz="0.08 -0 0.17" rpy="3.14159 -0 0"/>
+    <origin xyz="0.08 0 0.175" rpy="0 0 0"/>
     <parent link="base_link"/>
     <child link="lidar_link"/>

File: urdf/my_robot.urdf.xacro (robot description, xacro)
@@ -2,9 +2,10 @@
 <!-- Generated using onshape-to-robot -->
 <!-- Onshape document_id: 3023829f8e4e5c564f6b4985 -->
-<robot name="tretabot" xmlns:xacro="http://www.ros.org/wiki/xacro">
+<robot name="tetrabot" xmlns:xacro="http://www.ros.org/wiki/xacro">
     <xacro:include filename="xacro_properties/xacro_properties.xacro" />
     <xacro:include filename="modules/base_y_llantas.xacro" />
     <xacro:include filename="modules/camara.xacro" />
     <xacro:include filename="modules/lidar.xacro" />
+    <xacro:include filename="modules/accesorios.xacro" />
     <xacro:include filename="gazebo/gazebo_plugins.xacro" />
     <xacro:include filename="gazebo/gazebo_properties.xacro" />

File: urdf/xacro_properties/xacro_properties.xacro (robot description, xacro)
@@ -4,4 +4,4 @@
 <robot xmlns:xacro="http://www.ros.org/wiki/xacro">
 <xacro:property name="package_name" value="my_robot_description" />
-<xacro:property name="robot_name" value="tretabot" />
+<xacro:property name="robot_name" value="tetrabot" />
 </robot>
