Commit message: Corrige joint duplicado, actualiza xacros y añade modelos/mapas nuevos

File: urdf/modules/base_y_llantas.xacro (robot description, xacro)
@@ -11,19 +11,19 @@
       <origin xyz="0 0 0.0158450026" rpy="0 0 0" />
   </joint>
-  <!-- Link base_t -->
+<!-- Link base_link -->
   <link name="base_link">
     <inertial>
-      <origin xyz="0.0107572 -0.000338235 0.0779814" rpy="0 0 0"/>
-      <mass value="4.83557"/>
-      <inertia ixx="0.0260829" ixy="-0.000213984" ixz="-0.00395219" iyy="0.0299972" iyz="3.98093e-05" izz="0.0405276"/>
+      <origin xyz="0.0260294 -0.000407716 0.0619833" rpy="0 0 0"/>
+      <mass value="13.7409"/>
+      <inertia ixx="0.0784468" ixy="-0.000814426" ixz="-0.0136557" iyy="0.0940151" iyz="0.000209377" izz="0.106813"/>
     </inertial>
-    <!-- Part base_t -->
+    <!-- Part base_link -->
     <visual>
       <origin xyz="0 0 0" rpy="0 -0 0"/>
       <geometry>
-        <mesh filename="package://my_robot_description/assets/base_t.stl"/>
+        <mesh filename="package://my_robot_description/assets/base_link.stl"/>
       </geometry>
-      <material name="base_t_material">
-        <color rgba="0.537255 0.854902 0.827451 1"/>
+      <material name="base_link_material">
+        <color rgba="0.615686 0.811765 0.929412 1"/>
       </material>
     </visual>
@@ -31,5 +31,5 @@
       <origin xyz="0 0 0" rpy="0 -0 0"/>
       <geometry>
-        <mesh filename="package://my_robot_description/assets/base_t.stl"/>
+        <mesh filename="package://my_robot_description/assets/base_link.stl"/>
       </geometry>
     </collision>
@@ -38,11 +38,11 @@
   <link name="llanta_dere_del_link">
     <inertial>
-      <origin xyz="-0 -0 -0.0264625" rpy="0 0 0"/>
-      <mass value="0.0901579"/>
-      <inertia ixx="2.81915e-05" ixy="0" ixz="0" iyy="2.83576e-05" iyz="-0" izz="4.79296e-05"/>
+      <origin xyz="-0 0 -0.0264625" rpy="0 0 0"/>
+      <mass value="0.324568"/>
+      <inertia ixx="0.00010149" ixy="0" ixz="0" iyy="0.000102087" iyz="0" izz="0.000172547"/>
     </inertial>
     <!-- Part llanta_dere_del -->
     <visual>
-      <origin xyz="-0 0 -0.015" rpy="1.5708 0 0"/>
+      <origin xyz="0 0 -0.015" rpy="1.5708 -0 0"/>
       <geometry>
         <mesh filename="package://my_robot_description/assets/llanta_dere_del.stl"/>
@@ -53,5 +53,5 @@
     </visual>
     <collision>
-      <origin xyz="-0 0 -0.015" rpy="1.5708 0 0"/>
+      <origin xyz="0 0 -0.015" rpy="1.5708 -0 0"/>
       <geometry>
         <mesh filename="package://my_robot_description/assets/llanta_dere_del.stl"/>
@@ -59,7 +59,7 @@
     </collision>
   </link>
-  <!-- Joint from base_t to llanta_dere_del -->
+  <!-- Joint from base_link to llanta_dere_del -->
   <joint name="llanta_dere_del_joint" type="continuous">
-    <origin xyz="0.0441 -0.095 0.0162" rpy="-1.5708 0.765592 0"/>
+    <origin xyz="0.0441 -0.095 0.0162" rpy="-1.5708 -0 0"/>
     <parent link="base_link"/>
     <child link="llanta_dere_del_link"/>
@@ -70,11 +70,11 @@
   <link name="llanta_dere_tra_link">
     <inertial>
-      <origin xyz="-0 -0 -0.0264625" rpy="0 0 0"/>
-      <mass value="0.0901579"/>
-      <inertia ixx="2.81915e-05" ixy="0" ixz="0" iyy="2.83576e-05" iyz="0" izz="4.79296e-05"/>
+      <origin xyz="0 -0 -0.0264625" rpy="0 0 0"/>
+      <mass value="0.324568"/>
+      <inertia ixx="0.00010149" ixy="0" ixz="0" iyy="0.000102087" iyz="0" izz="0.000172547"/>
     </inertial>
     <!-- Part llanta_dere_tra -->
     <visual>
-      <origin xyz="-0 0 -0.015" rpy="1.5708 -0 0"/>
+      <origin xyz="0 -0 -0.015" rpy="1.5708 -0 0"/>
       <geometry>
         <mesh filename="package://my_robot_description/assets/llanta_dere_tra.stl"/>
@@ -85,5 +85,5 @@
     </visual>
     <collision>
-      <origin xyz="-0 0 -0.015" rpy="1.5708 -0 0"/>
+      <origin xyz="0 -0 -0.015" rpy="1.5708 -0 0"/>
       <geometry>
         <mesh filename="package://my_robot_description/assets/llanta_dere_tra.stl"/>
@@ -91,5 +91,5 @@
     </collision>
   </link>
-  <!-- Joint from base_t to llanta_dere_tra -->
+  <!-- Joint from base_link to llanta_dere_tra -->
   <joint name="llanta_dere_tra_joint" type="continuous">
     <origin xyz="-0.0859 -0.095 0.0162" rpy="-1.5708 -0 0"/>
@@ -103,6 +103,6 @@
     <inertial>
       <origin xyz="-0 0 -0.0264625" rpy="0 0 0"/>
-      <mass value="0.0901579"/>
-      <inertia ixx="2.81477e-05" ixy="0" ixz="0" iyy="2.84014e-05" iyz="0" izz="4.79296e-05"/>
+      <mass value="0.324568"/>
+      <inertia ixx="0.000101332" ixy="0" ixz="0" iyy="0.000102245" iyz="0" izz="0.000172547"/>
     </inertial>
     <!-- Part llanta_iz_del -->
@@ -123,5 +123,5 @@
     </collision>
   </link>
-  <!-- Joint from base_t to llanta_iz_del -->
+  <!-- Joint from base_link to llanta_iz_del -->
   <joint name="llanta_iz_del_joint" type="continuous">
     <origin xyz="0.0441 0.095 0.0162" rpy="1.5708 -0 0"/>
@@ -135,6 +135,6 @@
     <inertial>
       <origin xyz="0 0 -0.0264625" rpy="0 0 0"/>
-      <mass value="0.0901579"/>
-      <inertia ixx="2.81477e-05" ixy="0" ixz="0" iyy="2.84014e-05" iyz="0" izz="4.79296e-05"/>
+      <mass value="0.324568"/>
+      <inertia ixx="0.000101332" ixy="0" ixz="0" iyy="0.000102245" iyz="0" izz="0.000172547"/>
     </inertial>
     <!-- Part llanta_iz_tra -->
@@ -155,5 +155,5 @@
     </collision>
   </link>
-  <!-- Joint from base_t to llanta_iz_tra -->
+  <!-- Joint from base_link to llanta_iz_tra -->
   <joint name="llanta_iz_tra_joint" type="continuous">
     <origin xyz="-0.0859 0.095 0.0162" rpy="1.5708 -0 0"/>

File: urdf/modules/camara.xacro (robot description, xacro)
@@ -3,8 +3,8 @@
 <!-- Onshape document_id: 3023829f8e4e5c564f6b4985 -->
 <robot xmlns:xacro="http://www.ros.org/wiki/xacro">
-<!-- Link camara_t_s -->
+ <!-- Link camara_t_s -->
   <link name="camara_link">
     <inertial>
-      <origin xyz="-0 0 -0.00516528" rpy="0 0 0"/>
+      <origin xyz="0 0 -0.00516528" rpy="0 0 0"/>
       <mass value="0.0399941"/>
       <inertia ixx="6.59521e-06" ixy="0" ixz="0" iyy="6.59521e-06" iyz="0" izz="1.04207e-05"/>
@@ -12,5 +12,5 @@
     <!-- Part camara_t_s -->
     <visual>
-      <origin xyz="-0 0 0.005" rpy="3.14159 -0 1.5708"/>
+      <origin xyz="0 0 0.005" rpy="3.14159 -0 1.5708"/>
       <geometry>
         <mesh filename="package://my_robot_description/assets/camara_t_s.stl"/>
@@ -21,5 +21,5 @@
     </visual>
     <collision>
-      <origin xyz="-0 0 0.005" rpy="3.14159 -0 1.5708"/>
+      <origin xyz="0 0 0.005" rpy="3.14159 -0 1.5708"/>
       <geometry>
         <mesh filename="package://my_robot_description/assets/camara_t_s.stl"/>
@@ -27,7 +27,7 @@
     </collision>
   </link>
-  <!-- Joint from base_t to camara_t_s -->
+  <!-- Joint from base_link to camara_t_s -->
   <joint name="camara_joint" type="fixed">
-    <origin xyz="0.115 0 0.135" rpy=" 0 0 0 "/>
+    <origin xyz="0.115 0 0.13" rpy="0 0 0"/>
     <parent link="base_link"/>
     <child link="camara_link"/>

File: urdf/modules/lidar.xacro (robot description, xacro)
@@ -6,5 +6,5 @@
   <link name="lidar_link">
     <inertial>
-      <origin xyz="-0 0 -0.00994579" rpy="0 0 0"/>
+      <origin xyz="-0 -0 -0.00994579" rpy="0 0 0"/>
       <mass value="0.0591873"/>
       <inertia ixx="1.18545e-05" ixy="0" ixz="0" iyy="1.18545e-05" iyz="0" izz="1.49382e-05"/>
@@ -12,5 +12,5 @@
     <!-- Part lidar_t_s -->
     <visual>
-      <origin xyz="0 0 0.005" rpy="3.14159 -0 0"/>
+      <origin xyz="0 -0 0.005" rpy="3.14159 -0 0"/>
       <geometry>
         <mesh filename="package://my_robot_description/assets/lidar_t_s.stl"/>
@@ -21,5 +21,5 @@
     </visual>
     <collision>
-      <origin xyz="0 0 0.005" rpy="3.14159 -0 0"/>
+      <origin xyz="0 -0 0.005" rpy="3.14159 -0 0"/>
       <geometry>
         <mesh filename="package://my_robot_description/assets/lidar_t_s.stl"/>
@@ -27,7 +27,7 @@
     </collision>
   </link>
-  <!-- Joint from base_t to lidar_t_s -->
+  <!-- Joint from base_link to lidar_t_s -->
   <joint name="lidar_joint" type="fixed">
-    <origin xyz="0.08 0 0.175" rpy="0 0 0"/>
+    <origin xyz="0.08 0 0.17" rpy="0 0 0"/>
     <parent link="base_link"/>
     <child link="lidar_link"/>
